File: eagle-files/Board/pid_projekat.brd (EAGLE design)
At the start: 89.8 x 66 mm, 32 parts, among them IC1 ATmega 328p, IC2 L298, IC3 78L05Z, IC4 DIL4 8 MHz, IC5 MAX232, J1 DCJ0202, X1 22-23-2021

Commit message: 21-09-2015 backup
Parts:
- added C11, C12: 100nF, capacitor-wima:C2.5-3
- added R1, R4: 10k, eagle-ltspice:0204/7
- added TAST1, TAST2: (no value), switch-omron:B3F-10XX
- moved R3 40.4 mm to (0.00, -20.3), turned to 0 degrees
Connections:
- removed net N$14: IC1.12, JP2.12
- removed net N$16: IC1.13, JP2.13
- removed net N$18: JP1.4
- removed net N$19: IC1.16, JP1.13
- removed net N$20: IC1.15, JP1.14
- removed net N$5: IC1.4
- removed net N$6: IC1.5, JP2.5
- new net ADC_0: IC1.23, JP1.6
- new net PD6: C11.1, IC1.12, JP2.12, R3.1, TAST1.1, TAST1.2
- new net PD7: C12.1, IC1.13, JP2.13, R4.1, TAST2.1, TAST2.2
- net ENC_A: now also IC1.4
- net ENC_B: now also IC1.5, JP1.4, JP2.5
- net ENC_BINV: no longer IC1.23, JP1.6
- net GND: now also C11.2, C12.2, TAST1.3, TAST1.4, TAST2.3, TAST2.4
- net MOT1: now also IC1.16, JP1.13
- net MOT2: now also IC1.15, JP1.14
- net RST: now also R1.1; no longer R3.1
- net VCC: now also R1.2, R4.2
Routing:
- net PD7: track 0.00 -> 43.3 mm
- net N$16: track 43.3 -> 0.00 mm
- net N$20: track 42.0 -> 0.00 mm
- net MOT2: track 72.6 -> 114.6 mm
- net MOT1: track 60.4 -> 96.8 mm
- net N$19: track 36.4 -> 0.00 mm
- net PD6: track 0.00 -> 31.7 mm
- net N$14: track 31.7 -> 0.00 mm
- net N$6: track 20.0 -> 0.00 mm, vias 1 -> 0
- net ENC_B: track 27.6 -> 47.6 mm, vias 0 -> 1
- net ENC_BINV: track 49.8 -> 45.8 mm
