File: eagle-files/Board/pid_projekat.sch (EAGLE design)
At the start: 32 parts, among them IC1 ATmega 328p, IC2 L298, IC3 78L05Z, IC4 DIL4 8 MHz, IC5 MAX232, J1 DCJ0202, X1 22-23-2021

Commit message: 21-09-2015 backup
Parts:
- added C11, C12: 100nF, capacitor-wima:C2,5-3
- added R1, R4: 10k, eagle-ltspice:R0204/7
- added TAST1, TAST2: (no value), switch-omron:10-XX
Connections:
- removed net N$14: IC1.12, JP2.12
- removed net N$16: IC1.13, JP2.13
- removed net N$18: JP1.4
- removed net N$19: IC1.16, JP1.13
- removed net N$20: IC1.15, JP1.14
- removed net N$5: IC1.4
- removed net N$6: IC1.5, JP2.5
- new net ADC_0: IC1.23, JP1.6
- new net PD6: C11.1, IC1.12, JP2.12, R3.1, TAST1.S, TAST1.S1
- new net PD7: C12.1, IC1.13, JP2.13, R4.1, TAST2.S, TAST2.S1
- net ENC_A: now also IC1.4
- net ENC_B: now also IC1.5, JP1.4, JP2.5
- net ENC_BINV: no longer IC1.23, JP1.6
- net GND: now also C11.2, C12.2, TAST1.P, TAST1.P1, TAST2.P, TAST2.P1
- net MOT1: now also IC1.16, JP1.13
- net MOT2: now also IC1.15, JP1.14
- net RST: now also R1.1; no longer R3.1
- net VCC: now also R1.2, R4.2
Other:
- moved on the sheet: C7, C8, C9, IC5, R3
